File: kicad/ADC.kicad_pcb (KiCad board)
At the start: 2 copper layers, 50.8 x 27.5 mm, 43 parts, among them J2 Conn_01x02_Pin, J3 CJT-T-P-XX-RA-BH1, J4 Conn_01x03_Pin, J5 Conn_01x05_Pin, U1 ADA4945-1ACPZ-RL, U2 ADR4525, U3 ADA4807-1ARJZ-R2, U4 ADP7118AUJZ-3.3-R7, U6 ADP7118AUJZ-1.8-R7, U7 AD4001BRMZ

Commit message: Newest Hydrophone ADC board updates
Use mkdocs to render documentation locally
Parts:
- removed C4: 10uF, Capacitor_SMD:C_0603_1608Metric_Pad1.08x0.95mm_HandSolder
- removed J2: Conn_01x02_Pin, Connector_PinHeader_2.54mm:PinHeader_1x02_P2.54mm_Vertical
- removed JP5, JP6: SolderJumper_2_Open, Jumper:SolderJumper-2_P1.3mm_Open_RoundedPad1.0x1.5mm
- removed TP1: TestPoint, TestPoint:TestPoint_Pad_D1.5mm
- added C15: 10pF, Capacitor_SMD:C_0603_1608Metric_Pad1.08x0.95mm_HandSolder, F.Cu at (169.2, 66.0)
- added C18: 100uF, Capacitor_SMD:C_0603_1608Metric_Pad1.08x0.95mm_HandSolder, F.Cu at (156.4, 73.7)
- added C20: 100nF, Capacitor_SMD:C_0603_1608Metric_Pad1.08x0.95mm_HandSolder, F.Cu at (156.5, 69.8)
- added C21: 100uF, Capacitor_SMD:C_0603_1608Metric_Pad1.08x0.95mm_HandSolder, F.Cu at (167.7, 65.8)
- added C22: 100nF, Capacitor_SMD:C_0603_1608Metric_Pad1.08x0.95mm_HandSolder, F.Cu at (167.7, 68.7)
- added C23: 1uF, Capacitor_SMD:C_0603_1608Metric_Pad1.08x0.95mm_HandSolder, F.Cu at (166.8, 72.8)
- added C24: 10uF, Capacitor_SMD:C_0603_1608Metric_Pad1.08x0.95mm_HandSolder, F.Cu at (156.7, 66.9)
- added C25: 10uF, Capacitor_SMD:C_0603_1608Metric_Pad1.08x0.95mm_HandSolder, F.Cu at (165.0, 64.4)
- added C26: 1uF, Capacitor_SMD:C_0603_1608Metric_Pad1.08x0.95mm_HandSolder, F.Cu at (161.7, 65.2)
- added C27: 1uF, Capacitor_SMD:C_0603_1608Metric_Pad1.08x0.95mm_HandSolder, F.Cu at (156.6, 71.8)
- added C28: 10uF, Capacitor_SMD:C_0603_1608Metric_Pad1.08x0.95mm_HandSolder, F.Cu at (161.1, 61.8)
- added C29: 1uF, Capacitor_SMD:C_0603_1608Metric_Pad1.08x0.95mm_HandSolder, F.Cu at (164.3, 54.3)
- added C30: 10uF, Capacitor_SMD:C_0603_1608Metric_Pad1.08x0.95mm_HandSolder, F.Cu at (164.3, 52.7)
- added C31: 180pF, Capacitor_SMD:C_0603_1608Metric_Pad1.08x0.95mm_HandSolder, F.Cu at (159.4, 52.9)
- added C32: 10uF, Capacitor_SMD:C_0603_1608Metric_Pad1.08x0.95mm_HandSolder, F.Cu at (167.6, 70.3)
- added C33: 100pF, Capacitor_SMD:C_0603_1608Metric_Pad1.08x0.95mm_HandSolder, F.Cu at (154.3, 54.9)
- added C34: 0.1uF, Capacitor_SMD:C_0603_1608Metric_Pad1.08x0.95mm_HandSolder, F.Cu at (161.7, 53.1)
- added C35: 1nF, Capacitor_SMD:C_0603_1608Metric_Pad1.08x0.95mm_HandSolder, F.Cu at (170.3, 57.5)
- added C36: 240pF, Capacitor_SMD:C_0603_1608Metric_Pad1.08x0.95mm_HandSolder, F.Cu at (170.4, 54.1)
- added C37: 240pF, Capacitor_SMD:C_0603_1608Metric_Pad1.08x0.95mm_HandSolder, F.Cu at (170.4, 60.8)
- added C38: 7.5pF, Capacitor_SMD:C_0603_1608Metric_Pad1.08x0.95mm_HandSolder, F.Cu at (177.5, 54.2)
- added C39: 7.5pF, Capacitor_SMD:C_0603_1608Metric_Pad1.08x0.95mm_HandSolder, F.Cu at (177.5, 60.6)
- added C40: 10uF, Capacitor_SMD:C_0603_1608Metric_Pad1.08x0.95mm_HandSolder, F.Cu at (161.4, 49.5)
- added C41: 1pF, Capacitor_SMD:C_0603_1608Metric_Pad1.08x0.95mm_HandSolder, F.Cu at (188.8, 41.5)
- added C42: 1pF, Capacitor_SMD:C_0603_1608Metric_Pad1.08x0.95mm_HandSolder, F.Cu at (180.2, 47.0)
- added C43: 10uF, Capacitor_SMD:C_0603_1608Metric_Pad1.08x0.95mm_HandSolder, F.Cu at (152.6, 47.8)
- added C44: 10uF, Capacitor_SMD:C_0603_1608Metric_Pad1.08x0.95mm_HandSolder, F.Cu at (185.8, 69.4)
- added C45: 10uF, Capacitor_SMD:C_0603_1608Metric_Pad1.08x0.95mm_HandSolder, F.Cu at (186.2, 61.5)
- added C46: 100pF, Capacitor_SMD:C_0603_1608Metric_Pad1.08x0.95mm_HandSolder, F.Cu at (154.3, 59.8)
- added C47: 100pF, Capacitor_SMD:C_0603_1608Metric_Pad1.08x0.95mm_HandSolder, F.Cu at (155.2, 57.4)
- added J1: Conn_01x03_Pin, Connector_PinHeader_2.54mm:PinHeader_1x03_P2.54mm_Vertical, F.Cu at (157.9, 63.2)
- added J6: Conn_01x02_Pin, Connector_PinHeader_2.54mm:PinHeader_1x02_P2.54mm_Vertical, F.Cu at (176.8, 67.1)
- added J7: Conn_01x02_Pin, Connector_PinHeader_2.54mm:PinHeader_1x02_P2.54mm_Vertical, F.Cu at (168.6, 44.7)
- added JP10: SolderJumper_3_Open, Jumper:SolderJumper-3_P1.3mm_Open_RoundedPad1.0x1.5mm_NumberLabels, B.Cu at (156.2, 67.2)
- added JP11: SolderJumper_3_Open, Jumper:SolderJumper-3_P1.3mm_Open_RoundedPad1.0x1.5mm_NumberLabels, B.Cu at (156.9, 71.8)
- added JP9: SolderJumper_3_Open, Jumper:SolderJumper-3_P1.3mm_Open_RoundedPad1.0x1.5mm_NumberLabels, B.Cu at (163.4, 74.3)
- added R12: 100k, Resistor_SMD:R_0603_1608Metric_Pad0.98x0.95mm_HandSolder, F.Cu at (150.4, 55.6)
- added R13: 100k, Resistor_SMD:R_0603_1608Metric_Pad0.98x0.95mm_HandSolder, F.Cu at (150.4, 58.9)
- added R14: 143, Resistor_SMD:R_0603_1608Metric_Pad0.98x0.95mm_HandSolder, F.Cu at (167.9, 56.5)
- added R15: 143, Resistor_SMD:R_0603_1608Metric_Pad0.98x0.95mm_HandSolder, F.Cu at (165.3, 57.5)
- added R16: 10, Resistor_SMD:R_0603_1608Metric_Pad0.98x0.95mm_HandSolder, F.Cu at (152.8, 58.0)
- added R18: 10, Resistor_SMD:R_0603_1608Metric_Pad0.98x0.95mm_HandSolder, F.Cu at (152.8, 56.5)
- added U5: LTC6373IDFM-PBF, LTC6373IDFM-PBF:05-08-1791_ADI, F.Cu at (160.8, 57.5)
- added U8: LTC3265EFE-PBF, LTC3265EFE-PBF:FE_20_ADI, F.Cu at (162.1, 69.5)
- added U9: LTC6655BHMS8-1.25-PBF, LTC6655BHMS8-1.25-PB:MSOP-8_MS_LIT, F.Cu at (185.0, 65.4)
- C12, C2: value 100pF -> 120pF
- C14: value 330p -> 10pF
- C9: value 1uF -> 10uF
- R10, R11, R2, R7: value 1k -> 10k
- R5, R8: value 120 -> 200
- R6, R9: value 1k -> 62.5k
- U2: value ADR4525 -> LTC6655BHMS8-1.25-PBF; footprint Package_SO:SOIC-8_3.9x4.9mm_P1.27mm -> LTC6655BHMS8-1.25-PB:MSOP-8_MS_LIT
- U3: value ADA4807-1ARJZ-R2 -> ADP7118ARDZ-3.3; footprint ADA4807-1ARJZ-R2:RJ_6_ADI -> ADP7118ARDZ-3-3:RD-8-1_ADI
- U4: value ADP7118AUJZ-3.3-R7 -> ADP7118ARDZ-1.8; footprint ADP7118:UJ-5_ADI -> ADP7118ARDZ-1-8:RD-8-1_ADI
- U6: value ADP7118AUJZ-1.8-R7 -> LTC6655BHMS8-2.5-PBF; footprint ADP7118:UJ-5_ADI -> LTC6655BHMS8-1.25-PB:MSOP-8_MS_LIT
- moved R7 54.4 mm to (153.9, 68.2), turned to 90 degrees
- moved R6 48.6 mm to (154.0, 71.6), turned to 90 degrees
- moved JP4 48.2 mm to (182.6, 43.2), turned to 90 degrees
- moved C14 45.8 mm to (152.4, 71.6), turned to 90 degrees
- moved JP3 45.3 mm to (179.8, 44.5), turned to -90 degrees
- moved JP2 43.6 mm to (185.4, 39.9), turned to 180 degrees
- moved JP1 40.8 mm to (188.8, 37.9), turned to 180 degrees
- moved R10 37.1 mm to (170.2, 69.6), turned to -90 degrees
- moved R9 35.9 mm to (171.1, 66.0), turned to -90 degrees
- moved U3 33.7 mm to (194.3, 40.7), turned to 180 degrees
- moved R11 31.3 mm to (175.2, 58.3), turned to 180 degrees
- moved U6 29.8 mm to (194.8, 49.8), turned to -90 degrees
- moved C6 29.6 mm to (199.3, 39.1), turned to 90 degrees
- moved C9 28.5 mm to (195.4, 53.7), turned to 0 degrees
- moved C3 28.1 mm to (191.1, 47.1), turned to 0 degrees
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Connections:
- net Net-(U1-VOCM) renamed +1V25#2
- C14 pad 1: /Analog frontend/PREAMP_OUT -> +8V5LDO
- C14 pad 2: GND -> /ADJ+
- C6 pad 1: +3.3V -> +3V3
- C7 pad 1: Net-(U2-OUT) -> VCC
- C9 pad 1: VCC -> +2V5
- J3 pad 2: /TWINAX_N -> /TWINAX_P
- J4 pad 3: +3.3V -> +3V3
- J5 pad 2: /DSP block/CIPO -> /DSP block/CNV
- J5 pad 3: /DSP block/SCK -> /DSP block/CIPO
- J5 pad 4: /DSP block/COPI -> /DSP block/SCK
- J5 pad 5: /DSP block/CNV -> /DSP block/COPI
- R10 pad 1: /Analog frontend/PREAMP_OUT -> /ADJ-
- R10 pad 2: Net-(R10-Pad2) -> GND
- R11 pad 2: GND -> /Analog frontend/RC_F1_N
- R2 pad 2: /Analog frontend/PREAMP_OUT -> /Analog frontend/RC_F1_P
- R6 pad 1: Net-(U5--) -> +8V5LDO
- R6 pad 2: /TWINAX_N -> /ADJ+
- R7 pad 1: Net-(U5-+) -> /ADJ+
- R7 pad 2: /TWINAX_N -> GND
- R9 pad 1: Net-(R9-Pad1) -> -8V5LDO
- R9 pad 2: Net-(R9-Pad2) -> /ADJ-
- TP2 pad 1: +3.3V -> +3V3
- U2 pad 1: unconnected-(U2-NC-Pad1) -> VCC
- U2 pad 3: unconnected-(U2-NC-Pad3) -> GND
- U2 pad 5: unconnected-(U2-NC-Pad5) -> GND
- U2 pad 6: Net-(U2-OUT) -> +1V25
- U2 pad 7: unconnected-(U2-NC-Pad7) -> +1V25
- U2 pad 8: unconnected-(U2-NC-Pad8) -> GND
- U3 pad 1: +2V5 -> +3V3
- U3 pad 2: GND -> +3V3
- U3 pad 3: Net-(U2-OUT) -> +3V3
- U3 pad 4: +2V5 -> GND
- U3 pad 5: Net-(JP5-B) -> Net-(JP1-A)
- U3 pad 6: VCC -> Net-(U3-SS)
- U4 pad 1: VCC -> +1V8
- U4 pad 2: GND -> +1V8
- U4 pad 3: Net-(JP1-A) -> +1V8
- U4 pad 4: +3.3V -> GND
- U4 pad 5: +3.3V -> Net-(JP3-B)
- U6 pad 2: GND -> VCC
- U6 pad 3: Net-(JP3-B) -> GND
- U6 pad 4: +1V8 -> GND
- U6 pad 5: +1V8 -> GND
Routing:
- net (no net): track 60.7 -> 0.00 mm
- net VCC: track 77.4 -> 24.6 mm
- net Teensy_A2: track 0.00 -> 34.0 mm
- net -8V5LDO: track 0.00 -> 26.7 mm, vias 0 -> 3
- net +8V5LDO: track 0.00 -> 25.5 mm, vias 0 -> 2
- net +2V5: track 28.9 -> 4.46 mm
- net GND: track 25.9 -> 9.34 mm, vias 15 -> 62
- net +3V3: track 0.00 -> 12.3 mm
- net /Analog frontend/RC_F1_N: track 0.00 -> 11.9 mm
- net +3.3V: track 9.97 -> 0.00 mm, vias 2 -> 0
- net Net-(U5-IN+): track 0.00 -> 9.13 mm
- net +1V25: track 0.00 -> 9.11 mm
- net /ADJ-: track 0.00 -> 9.08 mm
- net Net-(U5-IN-): track 0.00 -> 8.93 mm
- net Net-(JP1-A): track 0.00 -> 8.60 mm
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- added copper zone on F.Cu, net VCC
Other:
- board size 50.8 x 27.5 mm -> 64.4 x 43.8 mm
- board text added: "A0"
- board text added: "A1"
- board text added: "A2"
- board text added: "C33"
- board text added: "C46"
- board text added: "C47"
- board text added: "GND VCC"
- board text added: "R12"
- board text added: "R13"
- board text added: "R16"
- board text added: "R18"
- board text added: "VCC VIO 3V3"
- board text removed: "3.3 VIO 5.0"
- board text removed: "VCC GND"

Commit message: updates
Parts:
- removed U5: LTC6373IDFM-PBF, LTC6373IDFM-PBF:05-08-1791_ADI
- added U10: LTC6373SDFM-PBF, LTC6373IDFM-PBF:05-08-1791_ADI, F.Cu at (160.8, 57.4)
- U3: footprint ADP7118ARDZ-3-3:RD-8-1_ADI -> ADP7118ARDZ-1-8:RD-8-1_ADI
- U6: footprint LTC6655BHMS8-1.25-PB:MSOP-8_MS_LIT -> LTC6655BHMS8-2.5-PB:MSOP-8_MS_LIT
- moved R14 3.98 mm to (164.3, 58.1), turned to -90 degrees
- moved R15 0.88 mm to (165.8, 56.9)
- moved C3 0.25 mm to (191.3, 47.1)
- moved C43 0.24 mm to (152.3, 47.9)
- moved U2 0.22 mm to (156.4, 49.5)
- moved U9 0.14 mm to (185.2, 65.4)
- moved U6 0.11 mm to (194.9, 49.7)
- moved U3 0.07 mm to (194.3, 40.6)
Connections:
- net Net-(U5-IN+) renamed /Analog frontend/PGA_IN_P
- net Net-(U5-IN-) renamed /Analog frontend/PGA_IN_N
Routing:
- net /Analog frontend/RC_F1_P: track 7.55 -> 12.7 mm
- net /Analog frontend/PREAMP_OUT_P: track 6.13 -> 2.46 mm
- net VCC: track 24.6 -> 26.7 mm
- net /Analog frontend/PREAMP_OUT_N: track 5.81 -> 3.95 mm
- net /Analog frontend/RC_F1_N: track 11.9 -> 10.9 mm

Commit message: added files for rev 1.1
Parts:
- removed U2: LTC6655BHMS8-1.25-PBF, LTC6655BHMS8-1.25-PB:MSOP-8_MS_LIT
- added U5: LTC6655CHMS8-1.25-PBF, LTC6655BHMS8-1.25-PB:MSOP-8_MS_LIT, F.Cu at (185.1, 65.5)
- C18, C21: footprint Capacitor_SMD:C_0603_1608Metric_Pad1.08x0.95mm_HandSolder -> Capacitor_SMD:C_1206_3216Metric_Pad1.33x1.80mm_HandSolder
- U9: value LTC6655BHMS8-1.25-PBF -> LTC6655CHMS8-1.25-PBF
- moved U9 32.7 mm to (156.6, 49.5), turned to 0 degrees
- moved C18 1.72 mm to (157.0, 75.3), turned to -90 degrees
- moved C21 0.97 mm to (167.3, 64.9)
- moved R9 0.36 mm to (171.4, 66.0)
- moved C44 0.18 mm to (185.8, 69.5)
- moved C45 0.17 mm to (186.2, 61.3)
Connections:
- U9 pad 6: +1V25#2 -> +1V25
- U9 pad 7: +1V25#2 -> +1V25
Routing:
- net GND: track 9.53 -> 26.5 mm, vias 62 -> 58
- net +1V25: track 9.11 -> 10.7 mm
- net VCC: track 26.7 -> 26.0 mm
- net /ADJ-: track 9.08 -> 9.72 mm
- net +8V5LDO: track 25.5 -> 26.0 mm
