File: kicad/ADC.kicad_sch (KiCad schematic)
At the start: 24 parts, among them J2 Conn_01x02_Pin, J3 CJT-T-P-XX-RA-BH1, J4 Conn_01x03_Pin, J5 Conn_01x05_Pin, U2 ADR4525, U3 ADA4807-1ARJZ-R2, U4 ADP7118AUJZ-3.3-R7, U6 ADP7118AUJZ-1.8-R7

Commit message: Newest Hydrophone ADC board updates
Use mkdocs to render documentation locally
Parts:
- removed C4: 10uF, Capacitor_SMD:C_0603_1608Metric_Pad1.08x0.95mm_HandSolder, symbol Device:C_US
- removed J2: Conn_01x02_Pin, Connector_PinHeader_2.54mm:PinHeader_1x02_P2.54mm_Vertical, symbol Connector:Conn_01x02_Pin
- removed JP5, JP6: SolderJumper_2_Open, Jumper:SolderJumper-2_P1.3mm_Open_RoundedPad1.0x1.5mm, symbol Jumper:SolderJumper_2_Open
- removed TP1: TestPoint, TestPoint:TestPoint_Pad_D1.5mm, symbol Connector:TestPoint
- removed U2: ADR4525, Package_SO:SOIC-8_3.9x4.9mm_P1.27mm, symbol Reference_Voltage:ADR4525
- removed U3: ADA4807-1ARJZ-R2, ADA4807-1ARJZ-R2:RJ_6_ADI, symbol ADA4807:ADA4807-1ARJZ-R2
- removed U4: ADP7118AUJZ-3.3-R7, UJ-5_ADI, symbol 3.3V LDO:ADP7118AUJZ-3.3-R7
- removed U6: ADP7118AUJZ-1.8-R7, UJ-5_ADI, symbol 1.8V LDO:ADP7118AUJZ-1.8-R7
- added C14, C15: 10pF, Capacitor_SMD:C_0603_1608Metric_Pad1.08x0.95mm_HandSolder, symbol Device:C
- added C18, C21: 100uF, Capacitor_SMD:C_0603_1608Metric_Pad1.08x0.95mm_HandSolder, symbol Device:C
- added C20, C22: 100nF, Capacitor_SMD:C_0603_1608Metric_Pad1.08x0.95mm_HandSolder, symbol Device:C
- added C23, C26: 1uF, Capacitor_SMD:C_0603_1608Metric_Pad1.08x0.95mm_HandSolder, symbol Device:C
- added C24, C25, C32: 10uF, Capacitor_SMD:C_0603_1608Metric_Pad1.08x0.95mm_HandSolder, symbol Device:C
- added C40, C43, C44, C45: 10uF, Capacitor_SMD:C_0603_1608Metric_Pad1.08x0.95mm_HandSolder, symbol Device:C_US
- added C41, C42: 1pF, Capacitor_SMD:C_0603_1608Metric_Pad1.08x0.95mm_HandSolder, symbol Device:C_US
- added J6, J7: Conn_01x02_Pin, Connector_PinHeader_2.54mm:PinHeader_1x02_P2.54mm_Vertical, symbol Connector:Conn_01x02_Pin
- added JP10, JP11, JP9: SolderJumper_3_Open, Jumper:SolderJumper-3_P1.3mm_Open_RoundedPad1.0x1.5mm_NumberLabels, symbol Jumper:SolderJumper_3_Open
- added R1: 1k, symbol Device:R
- added R10, R7: 10k, Resistor_SMD:R_0603_1608Metric_Pad0.98x0.95mm_HandSolder, symbol Device:R
- added R6, R9: 62.5k, Resistor_SMD:R_0603_1608Metric_Pad0.98x0.95mm_HandSolder, symbol Device:R
- added U2, U9: LTC6655BHMS8-1.25-PBF, LTC6655BHMS8-1.25-PB:MSOP-8_MS_LIT, symbol LTC6655-NR-1.25:LTC6655BHMS8-1.25-PBF
- added U3: ADP7118ARDZ-3.3, ADP7118ARDZ-3-3:RD-8-1_ADI, symbol 3.3V LDO (SOIC):ADP7118ARDZ-3.3
- added U4: ADP7118ARDZ-1.8, ADP7118ARDZ-1-8:RD-8-1_ADI, symbol 1.8V LDO (SOIC):ADP7118ARDZ-1.8
- added U6: LTC6655BHMS8-2.5-PBF, LTC6655BHMS8-1.25-PB:MSOP-8_MS_LIT, symbol LTC6655-NR-2.5:LTC6655BHMS8-2.5-PBF
- added U8: LTC3265EFE-PBF, LTC3265EFE-PBF:FE_20_ADI, symbol LTC3265:LTC3265EFE-PBF
- C9: value 1uF -> 10uF
Connections:
- net +1V8: now also U4.1 (VOUT), U4.2 (VOUT), U4.3 (SENSE/ADJ)
- net +2V5: now also C9.1, U6.6 (VOUT_S), U6.7 (VOUT_F)
- net DSP block/CIPO: now also J5.3 (Pin_3); no longer J5.2 (Pin_2)
- net DSP block/CNV: now also J5.2 (Pin_2); no longer J5.5 (Pin_5)
- net DSP block/COPI: now also J5.5 (Pin_5); no longer J5.4 (Pin_4)
- net DSP block/SCK: now also J5.4 (Pin_4); no longer J5.3 (Pin_3)
- net GND: now also C18.2, C20.2, C21.2, C22.2, C24.2, C25.2, C32.1, C40.2, C41.2, C42.2, C43.2, C44.2, C45.2, J6.1 (Pin_1), J7.1 (Pin_1), JP10.1 (A), JP11.1 (A), JP9.1 (A), R1.2, R10.2, R7.2, U2.3 (GND), U2.4 (GND), U2.5 (GND), U2.8 (GND), U3.4 (GND), U3.9 (GND), U4.4 (GND), U4.9 (GND), U6.3 (GND), U6.4 (GND), U6.5 (GND), U6.8 (GND), U8.EPAD, U9.3 (GND), U9.4 (GND), U9.5 (GND), U9.8 (GND)
- net TWINAX_N: now also J3.1; no longer J3.2
- net TWINAX_P: now also J3.2; no longer J3.1
- net VCC: now also C7.1, C32.2, C43.1, C44.1, J6.2 (Pin_2), J7.2 (Pin_2), JP10.3 (B), JP11.3 (B), JP9.3 (B), U2.1 (*SHDN), U2.2 (VIN), U3.7 (VIN), U3.8 (VIN), U4.7 (VIN), U4.8 (VIN), U6.1 (*SHDN), U6.2 (VIN), U8.4 (VINP), U9.1 (*SHDN), U9.2 (VIN); no longer C9.1
- net at JP3.2 (B), JP4.1 (A): now also U4.5 (EN)
- net at JP1.1 (A), JP2.1 (A): now also U3.5 (EN)
- net +3.3V renamed +3V3
- net +3V3: now also U3.1 (VOUT), U3.2 (VOUT), U3.3 (SENSE/ADJ)
- new net: C20.1, U8.17 (BYP+)
- new net: C42.1, U4.6 (SS)
- new net: C41.1, U3.6 (SS)
- new net: C22.1, U8.6 (BYP-)
- new net: C26.2, U8.10 (CINV)
- new net: R1.1, U8.14 (RT)
- new net: JP10.2 (C), U8.15 (EN+)
- new net: JP11.2 (C), U8.16 (MODE)
- new net: C23.1, U8.2 (CBST-)
- new net: C23.2, U8.3 (CBST+)
- new net: JP9.2 (C), U8.5 (EN-)
- new net: C25.1, U8.9 (VOUT-)
- new net: C26.1, U8.12 (CINV+)
- new net +1V25: C40.1, U2.6 (VOUT_S), U2.7 (VOUT_F)
- new net +1V25#2: C45.1, U9.6 (VOUT_S), U9.7 (VOUT_F)
- new net +8V5LDO: C14.1, C18.1, R6.1, U8.19 (LDO+)
- new net -8V5LDO: C15.1, C21.1, R9.1, U8.8 (LDO-)
- new net ADJ+: C14.2, R6.2, R7.1, U8.18 (ADJ+)
- new net ADJ-: C15.2, R10.1, R9.2, U8.7 (ADJ-)
- new net VOUT+: C24.1, U8.13 (VINN), U8.20 (VOUT+)
Other:
- note added: "(From datasheet) Connect *SHDWN pin at the load and route with a wide metal trace to minimize load regulation errors. This pin sinks 2mA"
- note added: "Equation for feedback network : V(LDO) = 1.2 * (R1/R2 + 1)"
- note added: "tying Vin_N to Vout+ will generate symetric power rails. The pump charge's positive and negative output voltages will be +/- 10V respectively. Since the boost charge pump generates 2*Vin_p on Vout+ and that the negative charge pump will also generate -Vout+ then the two charge pump outputs are +/-10V now"
- note removed: "2.5V voltage regulator"
- note removed: "mid-supply reference (VCC/2) for Vocm and ADC reference through voltage buffer"
- moved on the sheet: C3, C5, C6, C8, J3, J4, J5, JP1, JP2, JP3, JP4, TP2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

Commit message: updates
Parts:
- removed U2, U9: LTC6655BHMS8-1.25-PBF, LTC6655BHMS8-1.25-PB:MSOP-8_MS_LIT, symbol LTC6655-NR-1.25:LTC6655BHMS8-1.25-PBF
- removed U3: ADP7118ARDZ-3.3, ADP7118ARDZ-3-3:RD-8-1_ADI, symbol 3.3V LDO (SOIC):ADP7118ARDZ-3.3
- removed U4: ADP7118ARDZ-1.8, ADP7118ARDZ-1-8:RD-8-1_ADI, symbol 1.8V LDO (SOIC):ADP7118ARDZ-1.8
- removed U6: LTC6655BHMS8-2.5-PBF, LTC6655BHMS8-1.25-PB:MSOP-8_MS_LIT, symbol LTC6655-NR-2.5:LTC6655BHMS8-2.5-PBF
- added U2, U9: LTC6655BHMS8-1.25-PBF, LTC6655BHMS8-1.25-PB:MSOP-8_MS_LIT, symbol LTC6655-1.25:LTC6655BHMS8-1.25-PBF
- added U3: ADP7118ARDZ-3.3, ADP7118ARDZ-1-8:RD-8-1_ADI, symbol ADP7118ARDZ-3.3:ADP7118ARDZ-3.3
- added U4: ADP7118ARDZ-1.8, ADP7118ARDZ-1-8:RD-8-1_ADI, symbol ADP7118ARDZ-1.8:ADP7118ARDZ-1.8
- added U6: LTC6655BHMS8-2.5-PBF, LTC6655BHMS8-2.5-PB:MSOP-8_MS_LIT, symbol LTC6655-2.5:LTC6655BHMS8-2.5-PBF
Connections:
- net +1V25: now also U2.6 (VOUT_S), U2.7 (VOUT_F)
- net +1V25#2: now also U9.6 (VOUT_S), U9.7 (VOUT_F)
- net +1V8: now also U4.1 (VOUT), U4.2 (VOUT), U4.3 (SENSE/ADJ)
- net +2V5: now also U6.6 (VOUT_S), U6.7 (VOUT_F)
- net +3V3: now also U3.1 (VOUT), U3.2 (VOUT), U3.3 (SENSE/ADJ)
- net GND: now also U2.3 (GND), U2.4 (GND), U2.5 (GND), U2.8 (GND), U3.4 (GND), U3.9 (GND), U4.4 (GND), U4.9 (GND), U6.3 (GND), U6.4 (GND), U6.5 (GND), U6.8 (GND), U9.3 (GND), U9.4 (GND), U9.5 (GND), U9.8 (GND)
- net VCC: now also U2.1 (*SHDN), U2.2 (VIN), U3.7 (VIN), U3.8 (VIN), U4.7 (VIN), U4.8 (VIN), U6.1 (*SHDN), U6.2 (VIN), U9.1 (*SHDN), U9.2 (VIN)
- net at C42.1: now also U4.6 (SS)
- net at JP1.1 (A), JP2.1 (A): now also U3.5 (EN)
- net at C41.1: now also U3.6 (SS)
- net at JP3.2 (B), JP4.1 (A): now also U4.5 (EN)

Commit message: added files for rev 1.1
Parts:
- removed U2, U9: LTC6655BHMS8-1.25-PBF, LTC6655BHMS8-1.25-PB:MSOP-8_MS_LIT, symbol LTC6655-1.25:LTC6655BHMS8-1.25-PBF
- added U5, U9: LTC6655CHMS8-1.25-PBF, MSOP-8_MS_LIT, symbol LTC6655-1.25 revc:LTC6655CHMS8-1.25-PBF
- C18, C21: footprint Capacitor_SMD:C_0603_1608Metric_Pad1.08x0.95mm_HandSolder -> Capacitor_SMD:C_1206_3216Metric_Pad1.33x1.80mm_HandSolder
Connections:
- net +1V25: now also U9.6 (VOUT_S), U9.7 (VOUT_F)
- net +1V25#2: now also U5.6 (VOUT_S), U5.7 (VOUT_F)
- net GND: now also U5.3 (GND), U5.4 (GND), U5.5 (GND), U5.8 (GND), U9.3 (GND), U9.4 (GND), U9.5 (GND), U9.8 (GND)
- net VCC: now also U5.1 (*SHDN), U5.2 (VIN), U9.1 (*SHDN), U9.2 (VIN)
Other:
- note added: "NOTE: the initial component (LTC6655BHMS8-1.25) wasn't available anymore at AD so we used a pin to pin replacement (LTC6655CHMS8-1.25) that only has a different initial accuracy and temp. coefficient"
