File: kicad/analog.kicad_sch (KiCad schematic)
At the start: 19 parts, among them U1 ADA4945-1ACPZ-RL, U5 AD8421ARZ

Commit message: Newest Hydrophone ADC board updates
Use mkdocs to render documentation locally
Parts:
- removed C14: 330p, Capacitor_SMD:C_0603_1608Metric_Pad1.08x0.95mm_HandSolder, symbol Device:C_US
- removed R10, R6, R7, R9: 1k, Resistor_SMD:R_0603_1608Metric_Pad0.98x0.95mm_HandSolder, symbol Device:R
- removed U5: AD8421ARZ, symbol Amplifier_Instrumentation:AD8421ARZ
- added C27, C29: 1uF, Capacitor_SMD:C_0603_1608Metric_Pad1.08x0.95mm_HandSolder, symbol Device:C
- added C28, C30: 10uF, Capacitor_SMD:C_0603_1608Metric_Pad1.08x0.95mm_HandSolder, symbol Device:C
- added C31: 180pF, Capacitor_SMD:C_0603_1608Metric_Pad1.08x0.95mm_HandSolder, symbol Device:C
- added C33, C46, C47: 100pF, Capacitor_SMD:C_0603_1608Metric_Pad1.08x0.95mm_HandSolder, symbol Device:C
- added C34: 0.1uF, Capacitor_SMD:C_0603_1608Metric_Pad1.08x0.95mm_HandSolder, symbol Device:C_US
- added C35: 1nF, Capacitor_SMD:C_0603_1608Metric_Pad1.08x0.95mm_HandSolder, symbol Device:C
- added C36, C37: 240pF, Capacitor_SMD:C_0603_1608Metric_Pad1.08x0.95mm_HandSolder, symbol Device:C
- added C38, C39: 7.5pF, Capacitor_SMD:C_0603_1608Metric_Pad1.08x0.95mm_HandSolder, symbol Device:C
- added J1: Conn_01x03_Pin, Connector_PinHeader_2.54mm:PinHeader_1x03_P2.54mm_Vertical, symbol Connector:Conn_01x03_Pin
- added R12, R13: 100k, Resistor_SMD:R_0603_1608Metric_Pad0.98x0.95mm_HandSolder, symbol Device:R
- added R14, R15: 143, Resistor_SMD:R_0603_1608Metric_Pad0.98x0.95mm_HandSolder, symbol Device:R
- added R16, R18: 10, Resistor_SMD:R_0603_1608Metric_Pad0.98x0.95mm_HandSolder, symbol Device:R
- added U5: LTC6373IDFM-PBF, 05-08-1791_ADI, symbol LTC6373:LTC6373IDFM-PBF
- C12, C2: value 100pF -> 120pF
- R11, R2: value 1k -> 10k
- R5, R8: value 120 -> 200
Connections:
- net DIFF_IN_N: now also R13.1, R16.1
- net DRIV_IN_N: now also C39.2
- net DRIV_IN_P: now also C38.2
- net GND: now also C27.2, C28.2, C29.2, C30.2, C31.1, C33.1, C34.2, C36.2, C37.2, C46.2, R12.2, R13.2, U5.10 (GND); no longer R11.2
- net VCC: now also U5.5 (V+OUT)
- net at R3.2, U1.1 (-FB): now also C38.1
- net at R4.2, U1.4 (+FB): now also C39.1
- net +1V25#2: now reaches C13.1, U1.9 (VOCM)
- net PREAMP_OUT renamed RC_F1_P
- net RC_F1_P: now also C35.2, C36.1, R14.1
- new net: C46.1, C47.2, R16.2, U5.1 (IN-)
- new net: C33.2, C47.1, R18.2, U5.12 (IN+)
- new net: C31.2, U5.9 (CAP)
- new net +1V25: C34.1, U5.8 (VOCM)
- new net +8V5LDO: C27.1, C28.1, U5.4 (V+)
- new net -8V5LDO: C29.1, C30.1, U5.13 (V-)
- new net DIFF_IN_P: R12.1, R18.1
- new net PREAMP_OUT_N: R15.2, U5.7 (OUT-)
- new net PREAMP_OUT_P: R14.2, U5.6 (OUT+)
- new net RC_F1_N: C35.1, C37.1, R11.2, R15.1
- new net Teensy_A0: J1.1 (Pin_1), U5.3 (A1)
- new net Teensy_A1: J1.2 (Pin_2), U5.2 (A0-)
- new net Teensy_A2: J1.3 (Pin_3), U5.11 (A2)
Other:
- note added: "ADC Driver's role in the signal chain Second Order LPF Unity gain (for signal conditioning)"
- note added: "An FDA's FB is connected to its inputs in a closed loop manner So FB+ => IN- And FB- => IN+"
- note added: "Because the source hydrophone is low impedance only one bias current return R is needed, but I give the possibility to add two in case When using two Rs, make sure to keep a very low source imabalance as this could severely affect CMRRR"
- note added: "DC input bias current return"
- note added: "Differential gain of x10 What about termination / impedance matching ? DO THE THEVENIN EEQUIVALENT RESISTOR THING !!!"
- note added: "Gain selection (Teensy GPIO)"
- note added: "Input RC filter to minimize RFI rectification"
- note removed: "ADD A SECOND ORDER DIFFERENTIAL LPF here ! For anti aliasing Gain is 10k"
- note removed: "Differential gain of x10 What about termination / impedance matching ?"
- note removed: "fc​≈482 kHz"
- moved on the sheet: C1, C12, C13, C2, JP7, JP8, R11, R2, R3, R4, R5, R8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

Commit message: updates
Parts:
- removed U5: LTC6373IDFM-PBF, 05-08-1791_ADI, symbol LTC6373:LTC6373IDFM-PBF
- added U10: LTC6373SDFM-PBF, LTC6373IDFM-PBF:05-08-1791_ADI, symbol LTC6373:LTC6373SDFM-PBF
Connections:
- net +1V25: now also U10.8 (VOCM)
- net +8V5LDO: now also U10.4 (V+)
- net -8V5LDO: now also U10.13 (EPAD)
- net GND: now also U10.10 (DGND)
- net PREAMP_OUT_N: now also U10.7 (-OUT)
- net PREAMP_OUT_P: now also U10.6 (+OUT)
- net Teensy_A0: now also U10.3 (A1)
- net Teensy_A1: now also U10.2 (A0)
- net Teensy_A2: now also U10.11 (A2)
- net VCC: now also U10.5 (V+OUT)
- net PGA_IN_N: now reaches C46.1, C47.2, R16.2
- net PGA_IN_N: now also U10.1 (-IN)
- net PGA_IN_P: now reaches C33.2, C47.1, R18.2
- net PGA_IN_P: now also U10.12 (+IN)
- net at C31.2: now also U10.9 (CAP)
Other:
- note added: "EPAD is connected to V- (-8.5V)"
- moved on the sheet: C27, C28, C29, C30, C31, C34, J1
